Commit message: laser added

File: exp_assignment3/urdf/robot.xacro (robot description, xacro)
@@ -197,4 +197,32 @@
 	    <child link="camera_link"/>
   </joint>
+  <link name="hokuyo_link">
+	    <collision>
+	      <origin xyz="0 0 0.025" rpy="0 0 0"/>
+	      <geometry>
+		<box size="0.05 0.05 0.05"/>
+	      </geometry>
+	    </collision>
+	    <visual>
+	      <origin xyz="0 0 0.025" rpy="0 0 0"/>
+	      <geometry>
+		<box size="0.05 0.05 0.05"/>
+	      </geometry>
+	      <material name="red">
+		<color rgba="1 0 0 1"/>
+	      </material>
+	    </visual>
+	    <inertial>
+	      <mass value="1e-5" />
+	      <origin xyz="0 0 0" rpy="0 0 0"/>
+	      <inertia ixx="1e-6" ixy="0" ixz="0" iyy="1e-6" iyz="0" izz="1e-6" />
+	    </inertial>
+  </link>
+  <joint name="hokuyo_joint" type="fixed">
+	    <axis xyz="0 1 0" />
+	    <origin xyz="0.28 0 0.05" rpy="0 0 0"/>
+	    <parent link="link_chassis"/>
+	    <child link="hokuyo_link"/>
+	 </joint>
 <!--************************************TRANSMISSION****************************************-->
 <transmission name="head_joint_trans">

Commit message: all states implemented

File: exp_assignment3/urdf/robot.xacro (robot description, xacro)
@@ -163,8 +163,7 @@
   </link>
 <!--************************************JOINTS****************************************-->
-  <joint name="head_joint" type="revolute">
+  <joint name="head_joint" type="fixed">
   	<axis xyz="0 0 1"/>
-  	<limit effort="1000.0" lower="-3.14" upper="3.14" velocity="0.2"/>
-  	<origin rpy="0 0 0" xyz="0 0 0"/>
+	    <origin xyz="0 0 0" rpy="0 0 0"/>
   	<parent link="neck_link"/>
   	<child link="head_link"/>
@@ -192,5 +191,5 @@
   </joint>
   <joint name="camera_joint" type="fixed">
-	    <axis xyz="1 0 0" />
+	    <axis xyz="0 0 1" />
 	    <origin xyz="0 0 0" rpy="0 0 0"/>
 	    <parent link="head_link"/>
@@ -225,14 +224,3 @@
 	    <child link="hokuyo_link"/>
 	 </joint>
-<!--************************************TRANSMISSION****************************************-->
-<transmission name="head_joint_trans">
-	<type>transmission_interface/SimpleTransmission</type>
-	<joint name="head_joint">
-		<hardwareInterface>hardware_interface/EffortJointInterface</hardwareInterface>
-	</joint>
-	<actuator name="motor1">
-		<hardwareInterface>hardware_interface/EffortJointInterface</hardwareInterface>
-		<mechanicalInterface>1</mechanicalInterface>
-	</actuator>
-</transmission>
 </robot>
